Commit message: Added mimic joints in xacro, updated some xacro macro
Signed-off-by: Vittorio Lumare <vittorio.lumare@robotgarage.org>

File: yeah_hand_description/urdf/finger.xacro (robot description, xacro)
@@ -1,5 +1,5 @@
 <?xml version="1.0"?>
 <robot name="yeah_hand" xmlns:xacro="http://ros.org">
-<xacro:macro name="finger" params="prefix x_offset z_offset">
+<xacro:macro name="finger" params="prefix x_offset z_offset mimic_joint mcp_k pip_k dip_k">
   <link name="${prefix}_base">
     <visual>
@@ -43,4 +43,5 @@
     <axis xyz="1 0 0"/>
     <limit lower="-1.40" upper="0" effort="1.0" velocity="1.0"/>
+    <mimic joint="${mimic_joint}" multiplier="${mcp_k}" offset="0.0"/>
   </joint>
   <link name="${prefix}_medial">
@@ -65,4 +66,5 @@
     <axis xyz="1 0 0"/>
     <limit lower="-1.92" upper="0" effort="1.0" velocity="1.0"/>
+    <mimic joint="${mimic_joint}" multiplier="${pip_k}" offset="0.0"/>
   </joint>
   <link name="${prefix}_distal">
@@ -87,4 +89,5 @@
     <axis xyz="1 0 0"/>
     <limit lower="-0.8" upper="0" effort="1.0" velocity="1.0"/>
+    <mimic joint="${mimic_joint}" multiplier="${dip_k}" offset="0.0"/>
   </joint>
 </xacro:macro>

File: yeah_hand_description/urdf/servomotor.xacro (robot description, xacro)
@@ -1,6 +1,6 @@
 <?xml version="1.0"?>
 <robot name="yeah_hand" xmlns:xacro="http://ros.org">
-<xacro:macro name="fixed_component" params="component_name mesh_filename parent x y z roll pitch yaw">
-<link name="${component_name}">
+<xacro:macro name="servomotor" params="servo_name mesh_filename parent x y z roll pitch yaw">
+<link name="${servo_name}">
   <visual>
     <origin xyz="0 0 0" rpy="0 0 0"/>
@@ -17,8 +17,15 @@
   </collision>
 </link>
-<joint name="${component_name}_joint" type="fixed">
+<joint name="${servo_name}_fixed_joint" type="fixed">
   <parent link="${parent}"/>
-  <child link="${component_name}"/>
+  <child link="${servo_name}"/>
   <origin xyz="${x} ${y} ${z}" rpy="${roll} ${pitch} ${yaw}"/>
+</joint>
+<link name="${servo_name}_tendon"/>
+<joint name="${servo_name}_joint" type="revolute">
+  <parent link="${servo_name}"/>
+  <child link="${servo_name}_tendon"/>
+  <axis xyz="0 0 1"/>
+  <limit lower="0" upper="6.28" effort="1.0" velocity="1.0"/>
 </joint>
 </xacro:macro>

File: yeah_hand_description/urdf/thumb.xacro (robot description, xacro)
@@ -1,10 +1,10 @@
 <?xml version="1.0"?>
 <robot name="yeah_hand" xmlns:xacro="http://ros.org">
-<xacro:macro name="thumb" params="component_name mesh_filename parent x y z">
-<link name="${component_name}">
+<xacro:macro name="thumb" params="parent x y z mimic_joint mcp_k ip_k">
+<link name="thumb_base">
   <visual>
     <origin xyz="0 0 0" rpy="0 0 0"/>
     <geometry>
-      <mesh filename="package://yeah_hand_description/meshes/${mesh_filename}.dae"/>
+      <mesh filename="package://yeah_hand_description/meshes/Thumb Base.dae"/>
     </geometry>
     <material name="gray"/>
@@ -13,11 +13,11 @@
     <origin xyz="0 0 0" rpy="0 0 0"/>
     <geometry>
-      <mesh filename="package://yeah_hand_description/meshes/${mesh_filename}.dae"/>
+      <mesh filename="package://yeah_hand_description/meshes/Thumb Base.dae"/>
     </geometry>
   </collision>
 </link>
-<joint name="${component_name}_joint" type="revolute">
+<joint name="thumb_cmc_joint" type="revolute">
   <parent link="${parent}"/>
-  <child link="${component_name}"/>
+  <child link="thumb_base"/>
   <origin xyz="${x} ${y} ${z}" rpy="0 0 0"/>
   <axis xyz="0 0 1"/>
@@ -39,5 +39,5 @@
   </collision>
 </link>
-<joint name="thumb_proximal_joint" type="revolute">
+<joint name="thumb_mcp_joint" type="revolute">
   <parent link="thumb_base"/>
   <child link="thumb_proximal"/>
@@ -45,4 +45,5 @@
   <axis xyz="0 1 0"/>
   <limit lower="-1.409" upper="0" effort="1.0" velocity="1.0"/>
+  <mimic joint="${mimic_joint}" multiplier="${mcp_k}" offset="0"/>
 </joint>
 <link name="thumb_distal">
@@ -61,5 +62,5 @@
   </collision>
 </link>
-<joint name="thumb_distal_joint" type="revolute">
+<joint name="thumb_ip_joint" type="revolute">
   <parent link="thumb_proximal"/>
   <child link="thumb_distal"/>
@@ -67,4 +68,5 @@
   <axis xyz="0 1 0"/>
   <limit lower="-0.424" upper="0" effort="1.0" velocity="1.0"/>
+  <mimic joint="${mimic_joint}" multiplier="${ip_k}" offset="0"/>
 </joint>
 </xacro:macro>

File: yeah_hand_description/urdf/yeah_hand.xacro (robot description, xacro)
@@ -4,4 +4,5 @@
 <xacro:include filename="$(find yeah_hand_description)/urdf/finger.xacro" />
 <xacro:include filename="$(find yeah_hand_description)/urdf/thumb.xacro" />
+<xacro:include filename="$(find yeah_hand_description)/urdf/servomotor.xacro" />
   <material name="gray">
     <color rgba="0.7 0.7 0.7 1.0"/>
@@ -15,17 +16,17 @@
   <xacro:fixed_component component_name="trs_platform" mesh_filename="TRS Platform" parent = "skeleton" x="0" y="0" z="0" roll="0" pitch="0" yaw="0"/>
   <xacro:fixed_component component_name="thumb_rotation_servo" mesh_filename="WS-ST3215-Servomotor" parent = "skeleton" x="0.01875" y="0.002" z="0.1245" roll="0" pitch="0" yaw="0"/>
-  <xacro:thumb component_name="thumb_base" mesh_filename="Thumb Base" parent = "thumb_rotation_servo" x="0" y="0" z="-0.001"/>
+  <xacro:thumb parent = "thumb_rotation_servo" x="0" y="0" z="-0.001" mimic_joint="thumb_servo_joint" mcp_k="-0.227" ip_k="-0.0689"/>
   <!--  Other fingers  -->
-  <xacro:finger prefix="index" x_offset="0.0" z_offset="0.0" />
-  <xacro:finger prefix="middle" x_offset="-0.02" z_offset="0.0" />
-  <xacro:finger prefix="ring" x_offset="-0.041" z_offset="-0.004" />
-  <xacro:finger prefix="little" x_offset="-0.0635" z_offset="-0.014" />
+  <xacro:finger prefix="index" x_offset="0.0" z_offset="0.0" mimic_joint="index_servo_joint" mcp_k="-0.22" pip_k="-0.305" dip_k="-0.12"/>
+  <xacro:finger prefix="middle" x_offset="-0.02" z_offset="0.0" mimic_joint="middle_servo_joint" mcp_k="-0.22" pip_k="-0.305" dip_k="-0.12"/>
+  <xacro:finger prefix="ring" x_offset="-0.041" z_offset="-0.004" mimic_joint="ring_little_servo_joint" mcp_k="-0.22" pip_k="-0.305" dip_k="-0.12"/>
+  <xacro:finger prefix="little" x_offset="-0.0635" z_offset="-0.014" mimic_joint="ring_little_servo_joint" mcp_k="-0.22" pip_k="-0.305" dip_k="-0.12"/>
   <!--  Logic Board  -->
   <xacro:fixed_component component_name="logic_board" mesh_filename="WS-ESP32-Servo-Driver-Board" parent = "skeleton" x="0" y="0" z="0" roll="0" pitch="0" yaw="0" />
   <!--  Servos  -->
-  <xacro:fixed_component component_name="index_servo" mesh_filename="WS-ST3215-Servomotor" parent = "skeleton" x="0.0137" y="-0.016" z="0.0673" roll="-1.57" pitch="0" yaw="0" />
-  <xacro:fixed_component component_name="ring_servo" mesh_filename="WS-ST3215-Servomotor" parent = "skeleton" x="-0.0137" y="-0.016" z="0.0425" roll="-1.57" pitch="3.14" yaw="0" />
-  <xacro:fixed_component component_name="middle_servo" mesh_filename="WS-ST3215-Servomotor" parent = "skeleton" x="0.0137" y="-0.016" z="0.017" roll="-1.57" pitch="0" yaw="0" />
-  <xacro:fixed_component component_name="thumb_servo" mesh_filename="WS-ST3215-Servomotor" parent = "skeleton" x="-0.01107" y="-0.021" z="0.09025" roll="-1.57" pitch="1.57" yaw="0" />
+  <xacro:servomotor servo_name="index_servo" mesh_filename="WS-ST3215-Servomotor" parent = "skeleton" x="0.0137" y="-0.016" z="0.0673" roll="-1.57" pitch="0" yaw="0" />
+  <xacro:servomotor servo_name="ring_little_servo" mesh_filename="WS-ST3215-Servomotor" parent = "skeleton" x="-0.0137" y="-0.016" z="0.0425" roll="-1.57" pitch="3.14" yaw="0" />
+  <xacro:servomotor servo_name="middle_servo" mesh_filename="WS-ST3215-Servomotor" parent = "skeleton" x="0.0137" y="-0.016" z="0.017" roll="-1.57" pitch="0" yaw="0" />
+  <xacro:servomotor servo_name="thumb_servo" mesh_filename="WS-ST3215-Servomotor" parent = "skeleton" x="-0.01107" y="0.02" z="0.09025" roll="-1.57" pitch="1.57" yaw="3.14" />
   <!--  Covers  -->
   <xacro:fixed_component component_name="upper_cover" mesh_filename="Upper Cover" parent = "skeleton" x="0" y="0" z="0" roll="0" pitch="0" yaw="0"/>
