Commit message: updated urdf (thumb rotation joint)
Signed-off-by: Vittorio Lumare <vittorio.lumare@robotgarage.org>

File: yeah_hand_description/urdf/rotation_servomotor.xacro (robot description, xacro)
@@ -1,5 +1,5 @@
 <?xml version="1.0"?>
 <robot name="yeah_hand" xmlns:xacro="http://ros.org">
-<xacro:macro name="servomotor" params="servo_name mesh_filename parent x y z roll pitch yaw">
+<xacro:macro name="rotation_servomotor" params="servo_name mesh_filename parent x y z roll pitch yaw">
 <link name="${servo_name}">
   <visual>
@@ -22,10 +22,10 @@
   <origin xyz="${x} ${y} ${z}" rpy="${roll} ${pitch} ${yaw}"/>
 </joint>
-<link name="${servo_name}_tendon"/>
+<link name="${servo_name}_flange"/>
 <joint name="${servo_name}_joint" type="revolute">
   <parent link="${servo_name}"/>
-  <child link="${servo_name}_tendon"/>
+  <child link="${servo_name}_flange"/>
   <axis xyz="0 0 1"/>
-  <limit lower="0" upper="6.28" effort="1.0" velocity="1.0"/>
+  <limit lower="0" upper="1.57" effort="1.0" velocity="1.0"/>
 </joint>
 </xacro:macro>

File: yeah_hand_description/urdf/thumb.xacro (robot description, xacro)
@@ -17,10 +17,8 @@
   </collision>
 </link>
-<joint name="thumb_cmc_joint" type="revolute">
+<joint name="thumb_cmc_joint" type="fixed">
   <parent link="${parent}"/>
   <child link="thumb_base"/>
   <origin xyz="${x} ${y} ${z}" rpy="0 0 0"/>
-  <axis xyz="0 0 1"/>
-  <limit lower="0" upper="1.57" effort="1.0" velocity="1.0"/>
 </joint>
 <link name="thumb_proximal">

File: yeah_hand_description/urdf/yeah_hand.xacro (robot description, xacro)
@@ -1,8 +1,36 @@
 <?xml version="1.0"?>
 <robot name="yeah_hand" xmlns:xacro="http://ros.org">
+<ros2_control name="yeah_hand_system" type="system">
+  <hardware>
+    <plugin>yeah_hand_hardware/YeahHandSystem</plugin>
+<!--    <param name="some_param">value</param>-->
+    <!-- add your hardware params here -->
+  </hardware>
+  <joint name="index_servo_joint">
+    <command_interface name="position"/>
+    <state_interface name="position"/>
+  </joint>
+  <joint name="middle_servo_joint">
+    <command_interface name="position"/>
+    <state_interface name="position"/>
+  </joint>
+  <joint name="ring_little_servo_joint">
+    <command_interface name="position"/>
+    <state_interface name="position"/>
+  </joint>
+  <joint name="thumb_servo_joint">
+    <command_interface name="position"/>
+    <state_interface name="position"/>
+  </joint>
+  <joint name="thumb_rotation_servo_joint">
+    <command_interface name="position"/>
+    <state_interface name="position"/>
+  </joint>
+</ros2_control>
 <xacro:include filename="$(find yeah_hand_description)/urdf/fixed_component.xacro" />
 <xacro:include filename="$(find yeah_hand_description)/urdf/finger.xacro" />
 <xacro:include filename="$(find yeah_hand_description)/urdf/thumb.xacro" />
-<xacro:include filename="$(find yeah_hand_description)/urdf/servomotor.xacro" />
+<xacro:include filename="$(find yeah_hand_description)/urdf/flexion_servomotor.xacro" />
+<xacro:include filename="$(find yeah_hand_description)/urdf/rotation_servomotor.xacro" />
   <material name="gray">
     <color rgba="0.7 0.7 0.7 1.0"/>
@@ -15,6 +43,6 @@
   <!--  Thumb  -->
   <xacro:fixed_component component_name="trs_platform" mesh_filename="TRS Platform" parent = "skeleton" x="0" y="0" z="0" roll="0" pitch="0" yaw="0"/>
-  <xacro:fixed_component component_name="thumb_rotation_servo" mesh_filename="WS-ST3215-Servomotor" parent = "skeleton" x="0.01875" y="0.002" z="0.1245" roll="0" pitch="0" yaw="0"/>
-  <xacro:thumb parent = "thumb_rotation_servo" x="0" y="0" z="-0.001" mimic_joint="thumb_servo_joint" mcp_k="-0.227" ip_k="-0.0689"/>
+  <xacro:rotation_servomotor servo_name="thumb_rotation_servo" mesh_filename="WS-ST3215-Servomotor" parent = "skeleton" x="0.01875" y="0.002" z="0.1245" roll="0" pitch="0" yaw="0"/>
+  <xacro:thumb parent = "thumb_rotation_servo_flange" x="0" y="0" z="-0.001" mimic_joint="thumb_servo_joint" mcp_k="-0.227" ip_k="-0.0689"/>
   <!--  Other fingers  -->
   <xacro:finger prefix="index" x_offset="0.0" z_offset="0.0" mimic_joint="index_servo_joint" mcp_k="-0.22" pip_k="-0.305" dip_k="-0.12"/>
@@ -25,8 +53,8 @@
   <xacro:fixed_component component_name="logic_board" mesh_filename="WS-ESP32-Servo-Driver-Board" parent = "skeleton" x="0" y="0" z="0" roll="0" pitch="0" yaw="0" />
   <!--  Servos  -->
-  <xacro:servomotor servo_name="index_servo" mesh_filename="WS-ST3215-Servomotor" parent = "skeleton" x="0.0137" y="-0.016" z="0.0673" roll="-1.57" pitch="0" yaw="0" />
-  <xacro:servomotor servo_name="ring_little_servo" mesh_filename="WS-ST3215-Servomotor" parent = "skeleton" x="-0.0137" y="-0.016" z="0.0425" roll="-1.57" pitch="3.14" yaw="0" />
-  <xacro:servomotor servo_name="middle_servo" mesh_filename="WS-ST3215-Servomotor" parent = "skeleton" x="0.0137" y="-0.016" z="0.017" roll="-1.57" pitch="0" yaw="0" />
-  <xacro:servomotor servo_name="thumb_servo" mesh_filename="WS-ST3215-Servomotor" parent = "skeleton" x="-0.01107" y="0.02" z="0.09025" roll="-1.57" pitch="1.57" yaw="3.14" />
+  <xacro:flexion_servomotor servo_name="index_servo" mesh_filename="WS-ST3215-Servomotor" parent = "skeleton" x="0.0137" y="-0.016" z="0.0673" roll="-1.57" pitch="0" yaw="0" />
+  <xacro:flexion_servomotor servo_name="ring_little_servo" mesh_filename="WS-ST3215-Servomotor" parent = "skeleton" x="-0.0137" y="-0.016" z="0.0425" roll="-1.57" pitch="3.14" yaw="0" />
+  <xacro:flexion_servomotor servo_name="middle_servo" mesh_filename="WS-ST3215-Servomotor" parent = "skeleton" x="0.0137" y="-0.016" z="0.017" roll="-1.57" pitch="0" yaw="0" />
+  <xacro:flexion_servomotor servo_name="thumb_servo" mesh_filename="WS-ST3215-Servomotor" parent = "skeleton" x="-0.01107" y="0.02" z="0.09025" roll="-1.57" pitch="1.57" yaw="3.14" />
   <!--  Covers  -->
   <xacro:fixed_component component_name="upper_cover" mesh_filename="Upper Cover" parent = "skeleton" x="0" y="0" z="0" roll="0" pitch="0" yaw="0"/>
